File: TV-B-Gone.brd (EAGLE design)
At the start: 47.6 x 30.1 mm, 29 parts, among them IC1 ATTINY85V-10S

Commit message: small changes
Parts:
- removed C2: 100uF, rcl-ez:E2,5-5
- added C1: 100uF, SparkFun-Capacitors:PANASONIC_E
- moved C3 0.95 mm to (10.2, 21.3)
Connections:
- net GND: now also C1.-; no longer C2.-
- net VCC: now also C1.+; no longer C2.+
Routing:
- net VCC: track 106.2 -> 105.0 mm
Changed lines of the file:
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@@
 <setting verticaltext="up"/>
 </settings>
-<grid distance="0.0125" unitdist="inch" unit="inch" style="lines" multiple="1" display="no" altdistance="0.025" altunitdist="inch" altunit="inch"/>
+<grid distance="0.000000123031" unitdist="inch" unit="inch" style="lines" multiple="1" display="no" altdistance="0.025" altunitdist="inch" altunit="inch"/>
 <layers>
 <layer number="1" name="Top" color="4" fill="1" visible="yes" active="yes"/>
@@
 <attribute name="VALUE" x="29.718" y="19.7866" size="1.27" layer="27" ratio="10" rot="R180"/>
 </element>
-<element name="C2" library="rcl-ez" package="E2,5-5" value="100uF" x="9.144" y="27.051" smashed="yes">
-<attribute name="VALUE" x="11.557" y="24.638" size="1.27" layer="27" ratio="10"/>
-</element>
 <element name="LED5" library="minimidi" package="CHIPLED_1206" value="RED" x="4.826" y="22.606" smashed="yes" rot="R180">
 <attribute name="VALUE" x="2.921" y="24.257" size="1.27" layer="27" ratio="10" rot="R180"/>
@@
 <element name="R1" library="fab" package="R1206FAB" value="1K" x="10.16" y="15.24"/>
 <element name="R3" library="fab" package="R1206FAB" value="10K" x="10.16" y="17.78"/>
-<element name="C3" library="fab" package="C1206FAB" value="0.1uF" x="10.16" y="22.225"/>
+<element name="C3" library="fab" package="C1206FAB" value="0.1uF" x="10.16" y="21.2725"/>
 <element name="R5" library="fab" package="R1206FAB" value="10K (opt)" x="28.575" y="3.175" rot="R180"/>
 <element name="R2" library="fab" package="R1206FAB" value="0" x="25.690703125" y="10.1923125" rot="R90"/>
@@
 <element name="R10" library="fab" package="R1206FAB" value="0" x="37.7825" y="10.16" rot="R90"/>
 <element name="R11" library="fab" package="R1206FAB" value="0" x="37.7825" y="3.175" rot="R90"/>
+<element name="C1" library="SparkFun-Capacitors" package="PANASONIC_E" value="100uF" x="8.5725" y="26.67" rot="R180"/>
 </elements>
 <signals>
 <signal name="VCC">
 <contactref element="IC1" pad="8"/>
-<contactref element="C2" pad="+"/>
 <contactref element="LED5" pad="A"/>
 <contactref element="LED1" pad="A"/>
@@
 <wire x1="27.813" y1="15.642" x2="27.813" y2="13.8176" width="0.4064" layer="1"/>
 <wire x1="27.813" y1="13.8176" x2="29.1846" y2="12.446" width="0.4064" layer="1"/>
-<wire x1="7.874" y1="27.051" x2="4.995346875" y2="27.051" width="0.6096" layer="1"/>
 <wire x1="4.995346875" y1="27.051" x2="2.159" y2="27.051" width="0.6096" layer="1"/>
 <wire x1="2.159" y1="27.051" x2="2.032" y2="27.178" width="0.6096" layer="1"/>
@@
 <wire x1="4.826" y1="24.356" x2="7.394" y2="24.356" width="0.6096" layer="1"/>
 <wire x1="7.394" y1="24.356" x2="8.509" y2="23.241" width="0.6096" layer="1"/>
-<wire x1="8.509" y1="22.225" x2="8.509" y2="23.241" width="0.6096" layer="1"/>
+<wire x1="8.509" y1="21.2725" x2="8.509" y2="23.241" width="0.6096" layer="1"/>
 <wire x1="20.2565" y1="17.78" x2="20.2565" y2="19.1135" width="0.4064" layer="1"/>
 <wire x1="20.2565" y1="19.1135" x2="19.05" y2="20.32" width="0.4064" layer="1"/>
-<wire x1="8.509" y1="22.225" x2="8.509" y2="20.701" width="0.4064" layer="1"/>
-<wire x1="8.509" y1="20.701" x2="8.89" y2="20.32" width="0.4064" layer="1"/>
-<wire x1="8.89" y1="20.32" x2="14.605" y2="20.32" width="0.4064" layer="1"/>
-<wire x1="14.605" y1="20.32" x2="15.24" y2="20.955" width="0.4064" layer="1"/>
 <wire x1="4.826" y1="26.797" x2="4.826" y2="26.881653125" width="0.4064" layer="1"/>
 <wire x1="4.826" y1="26.881653125" x2="4.995346875" y2="27.051" width="0.4064" layer="1"/>
+<contactref element="C1" pad="+"/>
+<wire x1="8.509" y1="21.2725" x2="8.89" y2="21.2725" width="0.6096" layer="1"/>
+<wire x1="8.89" y1="21.2725" x2="10.7500875" y2="19.53083125" width="0.6096" layer="1"/>
+<wire x1="10.7500875" y1="19.53083125" x2="12.6550875" y2="19.53083125" width="0.6096" layer="1"/>
+<wire x1="12.6550875" y1="19.53083125" x2="14.2875" y2="20.955" width="0.6096" layer="1"/>
+<wire x1="14.2875" y1="20.955" x2="15.875" y2="20.955" width="0.6096" layer="1"/>
+<wire x1="5.5725" y1="26.67" x2="5.376346875" y2="26.67" width="0.6096" layer="1"/>
+<wire x1="5.376346875" y1="26.67" x2="4.995346875" y2="27.051" width="0.6096" layer="1"/>
 <wire x1="42.291" y1="20.066" x2="42.291" y2="20.066" width="0" layer="19" extent="1-16"/>
 <wire x1="42.291" y1="12.7" x2="42.291" y2="12.7" width="0" layer="19" extent="1-16"/>
-<wire x1="15.24" y1="20.955" x2="19.05" y2="20.32" width="0" layer="19" extent="1-1"/>
+<wire x1="15.875" y1="20.955" x2="19.05" y2="20.32" width="0" layer="19" extent="1-1"/>
 </signal>
 <signal name="GND">
 <contactref element="IC1" pad="4"/>
-<contactref element="C2" pad="-"/>
 <contactref element="-" pad="1"/>
 <polygon width="0.3048" layer="1" spacing="0.4064" isolate="0.635">
@@
 <contactref element="R10" pad="2"/>
 <contactref element="R11" pad="2"/>
+<contactref element="C1" pad="-"/>
 <wire x1="17.78" y1="10.541" x2="17.78" y2="7.239" width="0" layer="19" extent="1-1"/>
 <wire x1="37.7825" y1="4.826" x2="37.7825" y2="1.524" width="0" layer="19" extent="1-1"/>
